File: hardware/kicad/microgrid_48v.kicad_sch (KiCad schematic)
At the start: 90 parts, among them K1 Albright SW80B, Q1 CSD19536KCS, Q2 CSD19536KCS, Q3 CSD19536KCS, Q4 CSD19536KCS, Q5 CSD19536KCS, Q6 CSD19536KCS, Q7 CSD19536KCS, Q8 CSD19536KCS, U1 UCC27211A, U10 DC bus voltage front end, U11 Microgrid bus voltage front e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, U12 Utility-side voltage front end, U13 TMP235, U2 UCC27211A, U3 UCC27211A, U4 UCC27211A, U6 TMCS1123B2AQDVGRQ1, U7 TMCS1123B2AQDVGRQ1, U8 TMCS1123B2AQDVGRQ1, U9 PV voltage front end

Commit message: feat: define exact analog measurement front ends
Parts:
- U10: value DC bus voltage front end -> OPA320AQDBVRQ1G4
- U11: value Microgrid bus voltage front end -> AMC3330QDWERQ1 + OPA320
- U12: value Utility-side voltage front end -> AMC3330QDWERQ1 + OPA320
- U9: value PV voltage front end -> OPA320AQDBVRQ1G4
Changed lines of the file:
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@@
       (effects (font (size 1.27 1.27)))
     )
-    (property "Value" "PV voltage front end" (id 1) (at 493 749 0)
+    (property "Value" "OPA320AQDBVRQ1G4" (id 1) (at 493 749 0)
       (effects (font (size 1.27 1.27)))
     )
@@
       (effects (font (size 1.27 1.27)))
     )
-    (property "Value" "DC bus voltage front end" (id 1) (at 605 749 0)
+    (property "Value" "OPA320AQDBVRQ1G4" (id 1) (at 605 749 0)
       (effects (font (size 1.27 1.27)))
     )
@@
       (effects (font (size 1.27 1.27)))
     )
-    (property "Value" "Microgrid bus voltage front end" (id 1) (at 717 749 0)
+    (property "Value" "AMC3330QDWERQ1 + OPA320" (id 1) (at 717 749 0)
       (effects (font (size 1.27 1.27)))
     )
@@
       (effects (font (size 1.27 1.27)))
     )
-    (property "Value" "Utility-side voltage front end" (id 1) (at 829 749 0)
+    (property "Value" "AMC3330QDWERQ1 + OPA320" (id 1) (at 829 749 0)
       (effects (font (size 1.27 1.27)))
     )

Commit message: feat: expand complete analog front ends in schematic
Parts:
- removed JCOM: External RS485 A, symbol MG:JCOM
- removed KAC: G9KA-1A1B-E DC12, symbol MG:KAC
- removed Q2: CSD19536KCS, symbol MG:Q2
- removed RG3: 5R-15R tuning footprint, symbol MG:RG3
- removed RGS8: 5R-15R tuning footprint, symbol MG:RGS8
- removed RVL6: VOC divider lower resistor 4.99 kohm, symbol MG:RVL6
- added CU11DCL: 100 nF AMC3330 bypass, symbol MG:CU11DCL
- added CU11HLO100N: 100 nF AMC3330 bypass, symbol MG:CU11HLO100N
- added CU11HLO1N: 1 nF AMC3330 bypass, symbol MG:CU11HLO1N
- added CU11VDD1N: 1 nF AMC3330 bypass, symbol MG:CU11VDD1N
- added CU11VDD1U: 1 uF AMC3330 bypass, symbol MG:CU11VDD1U
- added CU12DCH1N: 1 nF AMC3330 bypass, symbol MG:CU12DCH1N
- added CU12DCH1U: 1 uF AMC3330 bypass, symbol MG:CU12DCH1U
- added CU12DCL: 100 nF AMC3330 bypass, symbol MG:CU12DCL
- added CU12HLO100N: 100 nF AMC3330 bypass, symbol MG:CU12HLO100N
- added CU12HLO1N: 1 nF AMC3330 bypass, symbol MG:CU12HLO1N
- added CU12IN: 1 nF isolated input filter, symbol MG:CU12IN
- added CU12VDD1N: 1 nF AMC3330 bypass, symbol MG:CU12VDD1N
- added CU12VDD1U: 1 uF AMC3330 bypass, symbol MG:CU12VDD1U
- added CU13: 100 nF TMP235 bypass, symbol MG:CU13
- added CU14: 100 nF local bypass, symbol MG:CU14
- added CU15: 100 nF local bypass, symbol MG:CU15
- added CUREF: 100 nF UREF bypass, symbol MG:CUREF
- added CUREF2: 100 nF UREF2 bypass, symbol MG:CUREF2
- added CVOC6: 10 uF threshold stabilizer, symbol MG:CVOC6
- added CVOC7: 10 uF threshold stabilizer, symbol MG:CVOC7
- added CVOC8: 10 uF threshold stabilizer, symbol MG:CVOC8
- added CVS6: 100 nF local supply bypass, symbol MG:CVS6
- added CVS7: 100 nF local supply bypass, symbol MG:CVS7
- added CVS8: 100 nF local supply bypass, symbol MG:CVS8
- added DK1: MURS120T3G, symbol MG:DK1
- added DKAC: MURS120T3G, symbol MG:DKAC
- added DKPRE: MURS120T3G, symbol MG:DKPRE
- added FBA: Analog rail ferrite input, symbol MG:FBA
- added JAC: Isolated grid emulator line, symbol MG:JAC
- added JBIAS: Gate-driver bias input, symbol MG:JBIAS
- added NTAGND: Analog/digital ground net tie, symbol MG:NTAGND
- added Q3: CSD19536KCS, symbol MG:Q3
- added Q7: CSD19536KCS, symbol MG:Q7
- added R165H: 10.0 kohm center-reference upper, symbol MG:R165H
- added R165L: 10.0 kohm center-reference lower, symbol MG:R165L
- added RDCH1: 100 kohm divider upper 1, symbol MG:RDCH1
- added RDCH2: 100 kohm divider upper 2, symbol MG:RDCH2
- added RDCL: 10.0 kohm divider lower, symbol MG:RDCL
- added RFDC: 1.00 kohm ADC isolation resistor, symbol MG:RFDC
- added RFPV: 1.00 kohm ADC isolation resistor, symbol MG:RFPV
- added RFTEMP: 1.00 kohm ADC isolation resistor, symbol MG:RFTEMP
- added RFU14: 1.00 kohm ADC isolation resistor, symbol MG:RFU14
- added RFU15: 1.00 kohm ADC isolation resistor, symbol MG:RFU15
- added RGS2: 5R-15R tuning footprint, symbol MG:RGS2
- added RPVH1: 100 kohm divider upper 1, symbol MG:RPVH1
- added RPVH2: 100 kohm divider upper 2, symbol MG:RPVH2
- added RPVL: 10.0 kohm divider lower, symbol MG:RPVL
- added RREFH: 30.4 kohm live-zero divider upper, symbol MG:RREFH
- added RREFL: 1.00 kohm live-zero divider lower, symbol MG:RREFL
- added RU11H1: 249 kohm isolation divider upper 1, symbol MG:RU11H1
- added RU11H2: 249 kohm isolation divider upper 2, symbol MG:RU11H2
- added RU11L: 10.0 kohm isolation divider shunt, symbol MG:RU11L
- added RU12H1: 249 kohm isolation divider upper 1, symbol MG:RU12H1
- added RU12L: 10.0 kohm isolation divider shunt, symbol MG:RU12L
- added RU14FB: 15.0 kohm feedback, symbol MG:RU14FB
- added RU14INN: 20.0 kohm difference input, symbol MG:RU14INN
- added RU14INP: 20.0 kohm difference input, symbol MG:RU14INP
- added RU14REF: 15.0 kohm reference leg, symbol MG:RU14REF
- added RU15FB: 15.0 kohm feedback, symbol MG:RU15FB
- added RU15INN: 20.0 kohm difference input, symbol MG:RU15INN
- added RU15INP: 20.0 kohm difference input, symbol MG:RU15INP
- added RU15REF: 15.0 kohm reference leg, symbol MG:RU15REF
- added RVH7: VOC divider upper resistor 8.40 kohm, symbol MG:RVH7
- added U13: TMP235, symbol MG:U13
- added U14: AMC3330 ADC driver, symbol MG:U14
- added U15: AMC3330 ADC driver, symbol MG:U15
- added U2: UCC27211A, symbol MG:U2
- added U8: TMCS1123B2AQDVGRQ1, symbol MG:U8
- added UEN4: PWM safety AND channel, symbol MG:UEN4
- added UREF: 105 mV reference buffer, symbol MG:UREF
- added UREF2: 1.65 V center-reference buffer, symbol MG:UREF2
- added URS485: ISO1410, symbol MG:URS485
- C165: renamed from CB1; value 100nF 50V C0G -> 100 nF center-reference filter; symbol MG:CB1 -> MG:C165
- CB1: renamed from CB2; symbol MG:CB2 -> MG:CB1
- CB2: renamed from CB3; symbol MG:CB3 -> MG:CB2
- CB3: renamed from CB4; symbol MG:CB4 -> MG:CB3
- CB4: renamed from CBULK6; symbol MG:CBULK6 -> MG:CB4
- CBULK6: renamed from CBULK7; symbol MG:CBULK7 -> MG:CBULK6
- CBULK7: renamed from CBULK8; symbol MG:CBULK8 -> MG:CBULK7
- CBULK8: renamed from CDC; value 3x ALS31A103KE100 -> 100nF 50V C0G; symbol MG:CDC -> MG:CBULK8
- CDC: renamed from CF; value C4AQUBW5200A3MJ 20uF -> 3x ALS31A103KE100; symbol MG:CF -> MG:CDC
- CF: renamed from CIN; value Input capacitor positive -> C4AQUBW5200A3MJ 20uF; symbol MG:CIN -> MG:CF
- CFDC: renamed from CVOC6; value 10 uF threshold stabilizer -> 4.7 nF ADC charge-bucket capacitor; symbol MG:CVOC6 -> MG:CFDC
- CFPV: renamed from CVOC7; value 10 uF threshold stabilizer -> 4.7 nF ADC charge-bucket capacitor; symbol MG:CVOC7 -> MG:CFPV
- CFTEMP: renamed from CVOC8; value 10 uF threshold stabilizer -> 4.7 nF ADC charge-bucket capacitor; symbol MG:CVOC8 -> MG:CFTEMP
- CFU14: renamed from CVS6; value 100 nF local supply bypass -> 4.7 nF ADC charge-bucket capacitor; symbol MG:CVS6 -> MG:CFU14
- CFU15: renamed from CVS7; value 100 nF local supply bypass -> 4.7 nF ADC charge-bucket capacitor; symbol MG:CVS7 -> MG:CFU15
- CIN: renamed from CVS8; value 100 nF local supply bypass -> Input capacitor positive; symbol MG:CVS8 -> MG:CIN
- CISO1410: renamed from DK1; value MURS120T3G -> 100 nF isolated RS-485 bypass; symbol MG:DK1 -> MG:CISO1410
- CREF: renamed from DKAC; value MURS120T3G -> 100 nF live-zero filter; symbol MG:DKAC -> MG:CREF
- CU10: renamed from F1; value JLLN030.T 30A -> 100 nF local bypass; symbol MG:F1 -> MG:CU10
- CU11DCH1N: renamed from JAC; value Isolated grid emulator line -> 1 nF AMC3330 bypass; symbol MG:JAC -> MG:CU11DCH1N
- CU11DCH1U: renamed from JBIAS; value Gate-driver bias input -> 1 uF AMC3330 bypass; symbol MG:JBIAS -> MG:CU11DCH1U
- CU11IN: renamed from JCTRL; value C2000 PWM output -> 1 nF isolated input filter; symbol MG:JCTRL -> MG:CU11IN
- CU9: renamed from DKPRE; value MURS120T3G -> 100 nF local bypass; symbol MG:DKPRE -> MG:CU9
- F1: renamed from Q3; value CSD19536KCS -> JLLN030.T 30A; symbol MG:Q3 -> MG:F1
- JCOM: renamed from Q7; value CSD19536KCS -> External RS485 A; symbol MG:Q7 -> MG:JCOM
- JCTRL: renamed from Q8; value CSD19536KCS -> C2000 PWM output; symbol MG:Q8 -> MG:JCTRL
- KAC: renamed from RGS2; value 5R-15R tuning footprint -> G9KA-1A1B-E DC12; symbol MG:RGS2 -> MG:KAC
- Q2: renamed from RVH7; value VOC divider upper resistor 8.40 kohm -> CSD19536KCS; symbol MG:RVH7 -> MG:Q2
- Q8: renamed from U2; value UCC27211A -> CSD19536KCS; symbol MG:U2 -> MG:Q8
- RG3: renamed from U8; value TMCS1123B2AQDVGRQ1 -> 5R-15R tuning footprint; symbol MG:U8 -> MG:RG3
- RGS8: renamed from U13; value TMP235 -> 5R-15R tuning footprint; symbol MG:U13 -> MG:RGS8
- RU12H2: renamed from UEN4; value PWM safety AND channel -> 249 kohm isolation divider upper 2; symbol MG:UEN4 -> MG:RU12H2
- RVL6: renamed from URS485; value ISO1410 -> VOC divider lower resistor 4.99 kohm; symbol MG:URS485 -> MG:RVL6
Connections:
- net 3V3: now also JCTRL.PWM1A, FBA.2, JBIAS.4, URS485.A; no longer CU11DCH1U.4, CU11IN.PWM1A, RGS8.OUT, RVL6.DE
- net 3V3_A: now also CBULK8.2, CU10.2, CU9.2, U10.IN-, U11.HLDO_OUT, U12.HLDO_OUT, U9.IN-, CU11VDD1N.2, CU11VDD1U.2, CU12VDD1N.2, CU12VDD1U.2, CU13.2, CU14.2, CU15.2, CUREF.2, CUREF2.2, CVS6.2, CVS7.2, CVS8.2, FBA.1, R165H.2, RREFH.2, U13.OUT, U14.IN-, U15.IN-, U8.GND, UREF.IN-, UREF2.IN-; no longer CB4.2, CFU14.2, CFU15.2, CIN.2, RG3.GND
- net 5V_ISO: now also CISO1410.2, JBIAS.5, URS485.DI; no longer CU11DCH1U.5, U10.IN-, U11.IN-, U12.IN-, U9.IN-
- net AC_INV: now also CF.2, RU11H1.2; no longer CDC.2, U11.GND
- net AC_PCC: now also KAC.COIL-, U8.ALERT; no longer RG3.ALERT
- net AC_RETURN: now also CB4.1, CU11DCH1U.1, CU11IN.1, Q8.G, U11.DCDC_GND, U11.GND, U11.OUTN, U12.DCDC_GND, U12.GND, U12.OUTN, CU11HLO100N.1, CU11HLO1N.1, CU12DCH1N.1, CU12DCH1U.1, CU12HLO100N.1, CU12HLO1N.1, CU12IN.1, JAC.1, Q7.S, RU11L.1, RU12L.1; no longer CB3.1, JCOM.S, JCTRL.G, U11.VCC, U12.VCC
- net ADC_GRID_I: now also JCTRL.ADC_GRID_I, U8.VOC; no longer CU11IN.ADC_GRID_I, RG3.VOC
- net ADC_GRID_V: now also CFU14.2, JCTRL.TRIP_LATCH_N, RFU14.1; no longer CU11IN.TRIP_LATCH_N, U11.OUT
- net ADC_IL_DC: now also JCTRL.ESTOP_N; no longer CU11IN.ESTOP_N
- net ADC_PV_I: now also JCTRL.PRECHARGE_CMD; no longer CU11IN.PRECHARGE_CMD
- net ADC_PV_V: now also CFPV.2, JCTRL.GRID_BREAKER_CMD, RFPV.1; no longer CU11IN.GRID_BREAKER_CMD, U9.OUT
- net ADC_TEMP: now also CFTEMP.2, JCTRL.ADC_UTILITY_V, RFTEMP.1; no longer CU11IN.ADC_UTILITY_V, RGS8.VCC
- net ADC_UTILITY_V: now also CFU15.2, JCTRL.ADC_TEMP, RFU15.1; no longer CU11IN.ADC_TEMP, U12.OUT
- net ADC_VDC: now also CFDC.2, JCTRL.MAIN_CONTACTOR_CMD, RFDC.1; no longer CU11IN.MAIN_CONTACTOR_CMD, U10.OUT
- net AGND: now also C165.1, CBULK8.1, CREF.1, CU10.1, CU9.1, RVL6.1, U10.IN+, U11.DCDC_HGND, U11.HGND, U12.DCDC_HGND, U12.HGND, U9.IN+, CU11DCL.1, CU11VDD1N.1, CU11VDD1U.1, CU12DCL.1, CU12VDD1N.1, CU12VDD1U.1, CU13.1, CU14.1, CU15.1, CUREF.1, CUREF2.1, CVOC6.1, CVOC7.1, CVOC8.1, CVS6.1, CVS7.1, CVS8.1, NTAGND.1, R165L.1, RREFL.1, U13.SENSE, U14.IN+, U15.IN+, U8.VS, UREF.IN+, UREF2.IN+; no longer CB4.1, CIN.1, RG3.VS
- net BIAS_POWER_GOOD: now also JCTRL.PWM4A, UEN4.ARM; no longer CU11IN.PWM4A, RU12H2.ARM
- net BOOT1+: now also CB1.2; no longer C165.2
- net BOOT2+: now also CB2.2, U2.HI; no longer CB1.2, Q8.HI
- net BOOT3+: now also CB3.2; no longer CB2.2
- net BOOT4+: now also CB4.2; no longer CB3.2
- net CF_DAMP: now also CF.1; no longer CDC.1
- net COM_GND_ISO: now also CISO1410.1, JCOM.1, URS485.RO; no longer RVL6.DI
- net DC48+: now also CDC.2, Q3.G, Q7.G, RDCH1.2; no longer CBULK8.2, F1.G, JCOM.G, U10.GND
- net DGND: now also JCTRL.PWM2A, JBIAS.2, NTAGND.2, URS485.DE; no longer CU11DCH1U.2, CU11IN.PWM2A, RGS8.SENSE, RVL6.RO, U10.IN+, U11.IN+, U12.IN+, U9.IN+
- net DRV_Q3: now also RG3.2, U2.VDD; no longer Q8.VDD
- net DRV_Q4: now also U2.HS; no longer Q8.HS
- net ESTOP_N: now also JCTRL.ADC_IL_DC, UTRIP.IN4_N, UEN4.TRIP_N; no longer CU11IN.ADC_IL_DC, RU12H2.TRIP_N, UTRIP.IN3_N
- net GATE_Q2: now also Q2.D, RGS2.2; no longer KAC.2
- net GATE_Q3: now also RG3.1, Q3.D; no longer F1.D
- net GATE_Q7: now also Q7.D; no longer JCOM.D
- net GATE_Q8: now also Q8.D, RGS8.2; no longer JCTRL.D
- net GD12V: now also JBIAS.6, U2.HO; no longer CU11DCH1U.6, Q8.HO
- net GRID_BREAKER_CMD: now also JCTRL.ADC_PV_V; no longer CU11IN.ADC_PV_V
- net GRID_COIL_LOW: now also KAC.COM, DKAC.K; no longer CREF.K
- net HEATSINK: now also U13.GND; no longer RGS8.GND
- net L2_RAW: now also U8.NC; no longer RG3.NC
- net MAIN_COIL_LOW: now also DK1.K; no longer CISO1410.K
- net MAIN_CONTACTOR_CMD: now also JCTRL.ADC_VDC; no longer CU11IN.ADC_VDC
- net OC_DC_N: now also UTRIP.DIAG_N; no longer UTRIP.OUT_N
- net OC_GRID_N: now also UTRIP.OUT_N, U8.VREF; no longer RG3.VREF, UTRIP.IN4_N
- net OC_PV_N: now also UTRIP.AFE_DIAG_N; no longer UTRIP.DIAG_N
- net PGND: now also CDC.1, CIN.1, JCTRL.PWM1B, Q2.S, Q8.S, RGS8.1, JBIAS.3, RGS2.1, U2.LI; no longer CBULK8.1, CF.1, CU11DCH1U.3, CU11IN.PWM1B, JCTRL.S, KAC.1, Q8.LI, U10.VCC, U9.VCC
- net PRECHARGE_CMD: now also JCTRL.ADC_PV_I; no longer CU11IN.ADC_PV_I
- net PRECHARGE_COIL_LOW: now also DKPRE.K; no longer CU9.K
- net PV_FUSED+: now also CIN.2, F1.1; no longer CF.2, CU10.1
- net PV_IN+: now also F1.2; no longer CU10.2
- net PV_SENSED+: now also RPVH1.2; no longer U9.GND
- net PWM1A_RAW: now also JCTRL.3V3; no longer CU11IN.3V3
- net PWM1B_RAW: now also JCTRL.PGND_SENSE; no longer CU11IN.PGND_SENSE
- net PWM2A: now also U2.HB; no longer Q8.HB
- net PWM2A_RAW: now also JCTRL.DGND; no longer CU11IN.DGND
- net PWM2B: now also U2.VSS, UEN4.PWM; no longer Q8.VSS, RU12H2.PWM
- net PWM2B_RAW: now also JCTRL.RS485_DE, UEN4.OUT; no longer CU11IN.RS485_DE, RU12H2.OUT
- net PWM3A_RAW: now also JCTRL.RS485_RX; no longer CU11IN.RS485_RX
- net PWM3B_RAW: now also JCTRL.RS485_TX; no longer CU11IN.RS485_TX
- net PWM4A_RAW: now also JCTRL.BIAS_POWER_GOOD; no longer CU11IN.BIAS_POWER_GOOD
- net PWM4B_RAW: now also JCTRL.PWM_ARM; no longer CU11IN.PWM_ARM
- net PWM_ARM: now also JCTRL.PWM4B, UEN4.BIAS_OK; no longer CU11IN.PWM4B, RU12H2.BIAS_OK
- net RELAY12V: now also KAC.NO, DK1.A, DKAC.A, DKPRE.A, JBIAS.1; no longer CISO1410.A, CREF.A, CU11DCH1U.1, CU9.A
- net RS485_A: now also JCOM.3, URS485.VCC; no longer RVL6.B
- net RS485_B: now also JCOM.2, URS485.B; no longer RVL6.A
- net RS485_DE: now also JCTRL.PWM2B, URS485.GND; no longer CU11IN.PWM2B, RVL6.VCC
- net RS485_RX: now also JCTRL.PWM3A, URS485.GND_ISO; no longer CU11IN.PWM3A, RVL6.GND
- net RS485_TX: now also JCTRL.PWM3B, URS485.VCC_ISO; no longer CU11IN.PWM3B, RVL6.GND_ISO
- net SENSOR_ALERT_N: now also UTRIP.IN2_N, U8.IP-; no longer RG3.IP-, UTRIP.IN1_N
- net SW_A: now also CB3.1; no longer CB2.1
- net SW_DC: now also CB2.1, Q3.S, U2.LO; no longer CB1.1, F1.S, Q8.LO
- net SW_PV: now also CB1.1, Q2.G; no longer C165.1
- net TRIP_LATCH_N: now also JCTRL.ADC_GRID_V, UTRIP.IN3_N, UEN4.ESTOP_N; no longer CU11IN.ADC_GRID_V, RU12H2.ESTOP_N, UTRIP.IN2_N
- net UTILITY_AC: now also KAC.COIL+, JAC.2, RU12H1.2; no longer CU11DCH1N.2, U12.GND
- net VOC_U6: now also RVL6.2, CVOC6.2; no longer CFDC.2
- net VOC_U7: now also CVOC7.2, RVH7.1; no longer CFPV.2, Q2.1
- net VOC_U8: now also CVOC8.2, U8.VOUT; no longer CFTEMP.2, RG3.VOUT
- net VREF_U7: now also RVH7.2; no longer Q2.2
- net VREF_U8: now also U8.OC; no longer RG3.OC
- new net AFE_DIAG_N: U11.HLDO_IN, U12.HLDO_IN, UTRIP.IN1_N
- new net DC_BUF: RFDC.2, U10.OUT, U10.VS
- new net DC_DIV: RDCH2.1, RDCL.2, U10.GND
- new net DC_DIV_MID: RDCH1.1, RDCH2.2
- new net PV_BUF: RFPV.2, U9.OUT, U9.VS
- new net PV_DIV: RPVH2.1, RPVL.2, U9.GND
- new net PV_DIV_MID: RPVH1.1, RPVH2.2
- new net TEMP_RAW: RFTEMP.2, U13.VS
- new net U11_DCDC_HI: CU11DCH1N.2, CU11DCH1U.2, U11.DCDC_IN, U11.DIAG
- new net U11_DCDC_LO: CU11DCL.2, U11.DCDC_OUT, U11.NC
- new net U11_DIV_MID: RU11H1.1, RU11H2.2
- new net U11_HLDO: CU11HLO100N.2, CU11HLO1N.2, U11.VDD
- new net U11_OUTN: RU14INN.2, U11.INN
- new net U11_OUTP: RU14INP.2, U11.INP
- new net U11_VSENSE: CU11IN.2, RU11H2.1, RU11L.2, U11.OUTP
- new net U12_DCDC_HI: CU12DCH1N.2, CU12DCH1U.2, U12.DCDC_IN, U12.DIAG
- new net U12_DCDC_LO: CU12DCL.2, U12.DCDC_OUT, U12.NC
- new net U12_DIV_MID: RU12H1.1, RU12H2.2
- new net U12_HLDO: CU12HLO100N.2, CU12HLO1N.2, U12.VDD
- new net U12_OUTN: RU15INN.2, U12.INN
- new net U12_OUTP: RU15INP.2, U12.INP
- new net U12_VSENSE: CU12IN.2, RU12H2.1, RU12L.2, U12.OUTP
- new net U14_NN: RU14FB.1, RU14INN.1, U14.VS
- new net U14_NP: RU14INP.1, RU14REF.1, U14.GND
- new net U14_OUT: RFU14.2, RU14FB.2, U14.OUT
- new net U15_NN: RU15FB.1, RU15INN.1, U15.VS
- new net U15_NP: RU15INP.1, RU15REF.1, U15.GND
- new net U15_OUT: RFU15.2, RU15FB.2, U15.OUT
- new net VREF105: RDCL.1, RPVL.1, UREF.OUT, UREF.VS
- new net VREF105_RAW: CREF.2, RREFH.1, RREFL.2, UREF.GND
- new net VREF165: RU14REF.2, RU15REF.2, UREF2.OUT, UREF2.VS
- new net VREF165_RAW: C165.2, R165H.1, R165L.2, UREF2.GND
- no-connect marks 3 -> 5
Other:
- moved on the sheet: JCOM
