File: hardware/kicad/microgrid_48v.kicad_sch (KiCad schematic)
At the start: 156 parts, among them K1 Albright SW80B, Q1 CSD19536KCS, Q2 CSD19536KCS, Q3 CSD19536KCS, Q4 CSD19536KCS, Q5 CSD19536KCS, Q6 CSD19536KCS, Q7 CSD19536KCS, Q8 CSD19536KCS, U1 UCC27211A, U10 OPA320AQDBVRQ1G4, U11 AMC3330QDWERQ1 + OPA320, U12 AMC3330QDWERQ1 + OPA320, U13 TMP235, U14 AMC3330 ADC driver, U15 AMC3330 ADC driver, U2 UCC27211A, U3 UCC27211A, U4 UCC27211A, U6 TMCS1123B2AQDVGRQ1, U7 TMCS1123B2AQDVGRQ1, U8 TMCS1123B2AQDVGRQ1, U9 OPA320AQDBVRQ1G4

Commit message: feat: assign frozen schematic footprints
Parts:
- Q1, Q2, Q3, Q4, Q5, Q6, Q7, Q8: footprint (none) -> Package_TO_SOT_THT:TO-220-3_Vertical
- U10, U14, U15, U9, UREF, UREF2: footprint (none) -> Package_TO_SOT_SMD:SOT-23-5
- U11, U12: footprint (none) -> Package_SO:SOIC-16W_7.5x10.3mm_P1.27mm
- U13: footprint (none) -> Package_TO_SOT_SMD:SOT-23
Changed lines of the file:
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@@
       (effects (font (size 1.27 1.27)))
     )
-    (property "Footprint" "" (id 2) (at 0 0 0)
-      (effects (font (size 1.27 1.27)) hide)
-    )
-    (property "Datasheet" "" (id 3) (at 0 0 0)
+    (property "Footprint" "Package_TO_SOT_THT:TO-220-3_Vertical" (id 2) (at 0 0 0)
+      (effects (font (size 1.27 1.27)) hide)
+    )
+    (property "Datasheet" "https://www.ti.com/lit/ds/symlink/csd19536kcs.pdf" (id 3) (at 0 0 0)
       (effects (font (size 1.27 1.27)) hide)
     )
@@
       (effects (font (size 1.27 1.27)))
     )
-    (property "Footprint" "" (id 2) (at 0 0 0)
-      (effects (font (size 1.27 1.27)) hide)
-    )
-    (property "Datasheet" "" (id 3) (at 0 0 0)
+    (property "Footprint" "Package_TO_SOT_THT:TO-220-3_Vertical" (id 2) (at 0 0 0)
+      (effects (font (size 1.27 1.27)) hide)
+    )
+    (property "Datasheet" "https://www.ti.com/lit/ds/symlink/csd19536kcs.pdf" (id 3) (at 0 0 0)
       (effects (font (size 1.27 1.27)) hide)
     )
@@
       (effects (font (size 1.27 1.27)))
     )
-    (property "Footprint" "" (id 2) (at 0 0 0)
-      (effects (font (size 1.27 1.27)) hide)
-    )
-    (property "Datasheet" "" (id 3) (at 0 0 0)
+    (property "Footprint" "Package_TO_SOT_THT:TO-220-3_Vertical" (id 2) (at 0 0 0)
+      (effects (font (size 1.27 1.27)) hide)
+    )
+    (property "Datasheet" "https://www.ti.com/lit/ds/symlink/csd19536kcs.pdf" (id 3) (at 0 0 0)
       (effects (font (size 1.27 1.27)) hide)
     )
@@
       (effects (font (size 1.27 1.27)))
     )
-    (property "Footprint" "" (id 2) (at 0 0 0)
-      (effects (font (size 1.27 1.27)) hide)
-    )
-    (property "Datasheet" "" (id 3) (at 0 0 0)
+    (property "Footprint" "Package_TO_SOT_THT:TO-220-3_Vertical" (id 2) (at 0 0 0)
+      (effects (font (size 1.27 1.27)) hide)
+    )
+    (property "Datasheet" "https://www.ti.com/lit/ds/symlink/csd19536kcs.pdf" (id 3) (at 0 0 0)
       (effects (font (size 1.27 1.27)) hide)
     )
@@
       (effects (font (size 1.27 1.27)))
     )
-    (property "Footprint" "" (id 2) (at 0 0 0)
-      (effects (font (size 1.27 1.27)) hide)
-    )
-    (property "Datasheet" "" (id 3) (at 0 0 0)
+    (property "Footprint" "Package_TO_SOT_THT:TO-220-3_Vertical" (id 2) (at 0 0 0)
+      (effects (font (size 1.27 1.27)) hide)
+    )
+    (property "Datasheet" "https://www.ti.com/lit/ds/symlink/csd19536kcs.pdf" (id 3) (at 0 0 0)
       (effects (font (size 1.27 1.27)) hide)
     )
@@
       (effects (font (size 1.27 1.27)))
     )
-    (property "Footprint" "" (id 2) (at 0 0 0)
-      (effects (font (size 1.27 1.27)) hide)
-    )
-    (property "Datasheet" "" (id 3) (at 0 0 0)
+    (property "Footprint" "Package_TO_SOT_THT:TO-220-3_Vertical" (id 2) (at 0 0 0)
+      (effects (font (size 1.27 1.27)) hide)
+    )
+    (property "Datasheet" "https://www.ti.com/lit/ds/symlink/csd19536kcs.pdf" (id 3) (at 0 0 0)
       (effects (font (size 1.27 1.27)) hide)
     )
@@
       (effects (font (size 1.27 1.27)))
     )
-    (property "Footprint" "" (id 2) (at 0 0 0)
-      (effects (font (size 1.27 1.27)) hide)
-    )
-    (property "Datasheet" "" (id 3) (at 0 0 0)
+    (property "Footprint" "Package_TO_SOT_THT:TO-220-3_Vertical" (id 2) (at 0 0 0)
+      (effects (font (size 1.27 1.27)) hide)
+    )
+    (property "Datasheet" "https://www.ti.com/lit/ds/symlink/csd19536kcs.pdf" (id 3) (at 0 0 0)
       (effects (font (size 1.27 1.27)) hide)
     )
@@
       (effects (font (size 1.27 1.27)))
     )
-    (property "Footprint" "" (id 2) (at 0 0 0)
-      (effects (font (size 1.27 1.27)) hide)
-    )
-    (property "Datasheet" "" (id 3) (at 0 0 0)
+    (property "Footprint" "Package_TO_SOT_THT:TO-220-3_Vertical" (id 2) (at 0 0 0)
+      (effects (font (size 1.27 1.27)) hide)
+    )
+    (property "Datasheet" "https://www.ti.com/lit/ds/symlink/csd19536kcs.pdf" (id 3) (at 0 0 0)
       (effects (font (size 1.27 1.27)) hide)
     )
@@
       (effects (font (size 1.27 1.27)) hide)
     )
-    (property "Datasheet" "" (id 3) (at 0 0 0)
+    (property "Datasheet" "https://www.ti.com/lit/ds/symlink/tmcs1123.pdf" (id 3) (at 0 0 0)
       (effects (font (size 1.27 1.27)) hide)
     )
@@
       (effects (font (size 1.27 1.27)) hide)
     )
-    (property "Datasheet" "" (id 3) (at 0 0 0)
+    (property "Datasheet" "https://www.ti.com/lit/ds/symlink/tmcs1123.pdf" (id 3) (at 0 0 0)
       (effects (font (size 1.27 1.27)) hide)
     )
@@
       (effects (font (size 1.27 1.27)) hide)
     )
-    (property "Datasheet" "" (id 3) (at 0 0 0)
+    (property "Datasheet" "https://www.ti.com/lit/ds/symlink/tmcs1123.pdf" (id 3) (at 0 0 0)
       (effects (font (size 1.27 1.27)) hide)
     )
@@
       (effects (font (size 1.27 1.27)))
     )
-    (property "Footprint" "" (id 2) (at 0 0 0)
-      (effects (font (size 1.27 1.27)) hide)
-    )
-    (property "Datasheet" "" (id 3) (at 0 0 0)
+    (property "Footprint" "Package_TO_SOT_SMD:SOT-23-5" (id 2) (at 0 0 0)
+      (effects (font (size 1.27 1.27)) hide)
+    )
+    (property "Datasheet" "https://www.ti.com/lit/ds/symlink/opa320-q1.pdf" (id 3) (at 0 0 0)
       (effects (font (size 1.27 1.27)) hide)
     )
@@
       (effects (font (size 1.27 1.27)))
     )
-    (property "Footprint" "" (id 2) (at 0 0 0)
-      (effects (font (size 1.27 1.27)) hide)
-    )
-    (property "Datasheet" "" (id 3) (at 0 0 0)
+    (property "Footprint" "Package_TO_SOT_SMD:SOT-23-5" (id 2) (at 0 0 0)
+      (effects (font (size 1.27 1.27)) hide)
+    )
+    (property "Datasheet" "https://www.ti.com/lit/ds/symlink/opa320-q1.pdf" (id 3) (at 0 0 0)
       (effects (font (size 1.27 1.27)) hide)
     )
@@
       (effects (font (size 1.27 1.27)))
     )
-    (property "Footprint" "" (id 2) (at 0 0 0)
-      (effects (font (size 1.27 1.27)) hide)
-    )
-    (property "Datasheet" "" (id 3) (at 0 0 0)
+    (property "Footprint" "Package_SO:SOIC-16W_7.5x10.3mm_P1.27mm" (id 2) (at 0 0 0)
+      (effects (font (size 1.27 1.27)) hide)
+    )
+    (property "Datasheet" "https://www.ti.com/lit/ds/symlink/amc3330-q1.pdf" (id 3) (at 0 0 0)
       (effects (font (size 1.27 1.27)) hide)
     )
@@
       (effects (font (size 1.27 1.27)))
     )
-    (property "Footprint" "" (id 2) (at 0 0 0)
-      (effects (font (size 1.27 1.27)) hide)
-    )
-    (property "Datasheet" "" (id 3) (at 0 0 0)
+    (property "Footprint" "Package_SO:SOIC-16W_7.5x10.3mm_P1.27mm" (id 2) (at 0 0 0)
+      (effects (font (size 1.27 1.27)) hide)
+    )
+    (property "Datasheet" "https://www.ti.com/lit/ds/symlink/amc3330-q1.pdf" (id 3) (at 0 0 0)
       (effects (font (size 1.27 1.27)) hide)
     )
@@
       (effects (font (size 1.27 1.27)))
     )
-    (property "Footprint" "" (id 2) (at 0 0 0)
-      (effects (font (size 1.27 1.27)) hide)
-    )
-    (property "Datasheet" "" (id 3) (at 0 0 0)
+    (property "Footprint" "Package_TO_SOT_SMD:SOT-23" (id 2) (at 0 0 0)
+      (effects (font (size 1.27 1.27)) hide)
+    )
+    (property "Datasheet" "https://www.ti.com/lit/ds/symlink/tmp235-q1.pdf" (id 3) (at 0 0 0)
       (effects (font (size 1.27 1.27)) hide)
     )
@@
       (effects (font (size 1.27 1.27)))
     )
-    (property "Footprint" "" (id 2) (at 0 0 0)
-      (effects (font (size 1.27 1.27)) hide)
-    )
-    (property "Datasheet" "" (id 3) (at 0 0 0)
+    (property "Footprint" "Package_TO_SOT_SMD:SOT-23-5" (id 2) (at 0 0 0)
+      (effects (font (size 1.27 1.27)) hide)
+    )
+    (property "Datasheet" "https://www.ti.com/lit/ds/symlink/opa320-q1.pdf" (id 3) (at 0 0 0)
       (effects (font (size 1.27 1.27)) hide)
     )
@@
       (effects (font (size 1.27 1.27)))
     )
-    (property "Footprint" "" (id 2) (at 0 0 0)
-      (effects (font (size 1.27 1.27)) hide)
-    )
-    (property "Datasheet" "" (id 3) (at 0 0 0)
+    (property "Footprint" "Package_TO_SOT_SMD:SOT-23-5" (id 2) (at 0 0 0)
+      (effects (font (size 1.27 1.27)) hide)
+    )
+    (property "Datasheet" "https://www.ti.com/lit/ds/symlink/opa320-q1.pdf" (id 3) (at 0 0 0)
       (effects (font (size 1.27 1.27)) hide)
     )
@@
       (effects (font (size 1.27 1.27)))
     )
-    (property "Footprint" "" (id 2) (at 0 0 0)
-      (effects (font (size 1.27 1.27)) hide)
-    )
-    (property "Datasheet" "" (id 3) (at 0 0 0)
+    (property "Footprint" "Package_TO_SOT_SMD:SOT-23-5" (id 2) (at 0 0 0)
+      (effects (font (size 1.27 1.27)) hide)
+    )
+    (property "Datasheet" "https://www.ti.com/lit/ds/symlink/opa320-q1.pdf" (id 3) (at 0 0 0)
       (effects (font (size 1.27 1.27)) hide)
     )
@@
       (effects (font (size 1.27 1.27)))
     )
-    (property "Footprint" "" (id 2) (at 0 0 0)
-      (effects (font (size 1.27 1.27)) hide)
-    )
-    (property "Datasheet" "" (id 3) (at 0 0 0)
-      (effects (font (size 1.27 1.27)) hide)
-    )
+    (property "Footprint" "Package_TO_SOT_SMD:SOT-23-5" (id 2) (at 0 0 0)
+      (effects (font (size 1.27 1.27)) hide)
+    )
+    (property "Datasheet" "https://www.ti.com/lit/ds/symlink/opa320-q1.pdf" (id 3) (at 0 0 0)
+      (effects (font (size 1.27 1.27)) hide)
+    )

Commit message: feat: assign reviewed signal-component footprints
Parts:
- C165, CFDC, CFPV, CFTEMP, CFU14, CFU15, CISO1410, CREF, CU10, CU11DCH1N, CU11DCH1U, CU11DCL, CU11HLO100N, CU11HLO1N, CU11IN, CU11VDD1N, CU11VDD1U, CU12DCH1N, CU12DCH1U, CU12DCL, CU12HLO100N, CU12HLO1N, CU12IN, CU12VDD1N, CU12VDD1U, CU13, CU14, CU15, CU9, CUREF, CUREF2, CVS6, CVS7, CVS8: footprint (none) -> Capacitor_SMD:C_0603_1608Metric_Pad1.08x0.95mm_HandSolder
- CB1, CB2, CB3, CB4, CBULK6, CBULK7, CBULK8, CVOC6, CVOC7, CVOC8: footprint (none) -> Capacitor_SMD:C_1206_3216Metric_Pad1.33x1.80mm_HandSolder
- DK1, DKAC, DKPRE: footprint (none) -> Diode_SMD:D_SMA
- FBA: footprint (none) -> Inductor_SMD:L_0603_1608Metric_Pad1.08x0.95mm_HandSolder
- NTAGND: footprint (none) -> NetTie:NetTie-2_SMD_Pad0.5mm
- QK1, QKAC, QKPRE: footprint (none) -> Package_TO_SOT_SMD:SOT-23
- R165H, R165L, RDCL, RFDC, RFPV, RFTEMP, RFU14, RFU15, RPVL, RREFH, RREFL, RU11L, RU12L, RU14FB, RU14INN, RU14INP, RU14REF, RU15FB, RU15INN, RU15INP, RU15REF, RVH6, RVH7, RVH8, RVL6, RVL7, RVL8: footprint (none) -> Resistor_SMD:R_0603_1608Metric_Pad0.98x0.95mm_HandSolder
- RDCH1, RDCH2, RPVH1, RPVH2, RU11H1, RU11H2, RU12H1, RU12H2: footprint (none) -> Resistor_SMD:R_1206_3216Metric_Pad1.42x1.75mm_HandSolder
- RG1, RG2, RG3, RG4, RG5, RG6, RG7, RG8, RGS1, RGS2, RGS3, RGS4, RGS5, RGS6, RGS7, RGS8: footprint (none) -> Resistor_SMD:R_0805_2012Metric_Pad1.20x1.40mm_HandSolder

Commit message: feat: complete C2000 Driverlib HAL, KiCad footprints, and Gate 2 design review
Parts:
- U1, U2, U3, U4: value UCC27211A -> UCC27211AQDDARQ1; footprint (none) -> Package_SO:SOIC-8-1EP_3.9x4.9mm_P1.27mm_EP2.95x3.4mm
- U6, U7, U8: footprint (none) -> Microgrid_48V:DVG0010A_HV
Connections:
- net 3V3_A: now also U6.3 (GND), U7.3 (GND), U8.3 (GND); no longer U6.GND, U7.GND, U8.GND
- net AC_PCC: now also U8.4 (ALERT); no longer U8.ALERT
- net AC_RETURN: now also U4.8 (LO); no longer U4.LO
- net ADC_GRID_I: now also U8.9 (VOC); no longer U8.VOC
- net ADC_IL_DC: now also U7.9 (VOC); no longer U7.VOC
- net ADC_PV_I: now also U6.9 (VOC); no longer U6.VOC
- net AGND: now also U6.8 (VS), U7.8 (VS), U8.8 (VS); no longer U6.VS, U7.VS, U8.VS
- net BOOT1+: now also U1.5 (HI); no longer U1.HI
- net BOOT2+: now also U2.5 (HI); no longer U2.HI
- net BOOT3+: now also U3.5 (HI); no longer U3.HI
- net BOOT4+: now also U4.5 (HI); no longer U4.HI
- net DRV_Q1: now also U1.1 (VDD); no longer U1.VDD
- net DRV_Q2: now also U1.4 (HS); no longer U1.HS
- net DRV_Q3: now also U2.1 (VDD); no longer U2.VDD
- net DRV_Q4: now also U2.4 (HS); no longer U2.HS
- net DRV_Q5: now also U3.1 (VDD); no longer U3.VDD
- net DRV_Q6: now also U3.4 (HS); no longer U3.HS
- net DRV_Q7: now also U4.1 (VDD); no longer U4.VDD
- net DRV_Q8: now also U4.4 (HS); no longer U4.HS
- net GD12V: now also U1.3 (HO), U2.3 (HO), U3.3 (HO), U4.3 (HO); no longer U1.HO, U2.HO, U3.HO, U4.HO
- net L2_RAW: now also U8.10 (NC); no longer U8.NC
- net LDC_RAW: now also U7.10 (NC); no longer U7.NC
- net OC_DC_N: now also U7.5 (VREF); no longer U7.VREF
- net OC_GRID_N: now also U8.5 (VREF); no longer U8.VREF
- net OC_PV_N: now also U6.5 (VREF); no longer U6.VREF
- net PGND: now also U1.6 (LI), U2.6 (LI), U3.6 (LI), U4.6 (LI); no longer U1.LI, U2.LI, U3.LI, U4.LI
- net PV_FUSED+: now also U6.10 (NC); no longer U6.NC
- net PV_SENSED+: now also U6.4 (ALERT); no longer U6.ALERT
- net PWM1A: now also U1.2 (HB); no longer U1.HB
- net PWM1B: now also U1.7 (VSS); no longer U1.VSS
- net PWM2A: now also U2.2 (HB); no longer U2.HB
- net PWM2B: now also U2.7 (VSS); no longer U2.VSS
- net PWM3A: now also U3.2 (HB); no longer U3.HB
- net PWM3B: now also U3.7 (VSS); no longer U3.VSS
- net PWM4A: now also U4.2 (HB); no longer U4.HB
- net PWM4B: now also U4.7 (VSS); no longer U4.VSS
- net SENSOR_ALERT_N: now also U6.2 (IP-), U7.2 (IP-), U8.2 (IP-); no longer U6.IP-, U7.IP-, U8.IP-
- net SW_A: now also U3.8 (LO); no longer U3.LO
- net SW_DC: now also U2.8 (LO), U7.4 (ALERT); no longer U2.LO, U7.ALERT
- net SW_PV: now also U1.8 (LO); no longer U1.LO
- net VOC_U6: now also U6.6 (VOUT); no longer U6.VOUT
- net VOC_U7: now also U7.6 (VOUT); no longer U7.VOUT
- net VOC_U8: now also U8.6 (VOUT); no longer U8.VOUT
- net VREF_U6: now also U6.7 (OC); no longer U6.OC
- net VREF_U7: now also U7.7 (OC); no longer U7.OC
- net VREF_U8: now also U8.7 (OC); no longer U8.OC
Other:
- moved on the sheet: U6, U7, U8
Changed lines of the file:
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@@
       (effects (font (size 1.27 1.27)))
     )
-    (property "Value" "UCC27211A" (id 1) (at 1053 1239 0)
-      (effects (font (size 1.27 1.27)))
-    )
-    (property "Footprint" "" (id 2) (at 0 0 0)
-      (effects (font (size 1.27 1.27)) hide)
-    )
-    (property "Datasheet" "" (id 3) (at 0 0 0)
-      (effects (font (size 1.27 1.27)) hide)
-    )
-    (pin "HI")
-    (pin "LI")
-    (pin "HO")
-    (pin "LO")
-    (pin "HS")
-    (pin "VDD")
-    (pin "VSS")
-    (pin "HB")
+    (property "Value" "UCC27211AQDDARQ1" (id 1) (at 1053 1239 0)
+      (effects (font (size 1.27 1.27)))
+    )
+    (property "Footprint" "Package_SO:SOIC-8-1EP_3.9x4.9mm_P1.27mm_EP2.95x3.4mm" (id 2) (at 0 0 0)
+      (effects (font (size 1.27 1.27)) hide)
+    )
+    (property "Datasheet" "https://www.ti.com/lit/ds/symlink/ucc27211a-q1.pdf" (id 3) (at 0 0 0)
+      (effects (font (size 1.27 1.27)) hide)
+    )
+    (pin "5")
+    (pin "6")
+    (pin "3")
+    (pin "8")
+    (pin "4")
+    (pin "1")
+    (pin "7")
+    (pin "2")
     (instances
       (project "microgrid_48v"
@@
       (effects (font (size 1.27 1.27)))
     )
-    (property "Value" "UCC27211A" (id 1) (at 45 1337 0)
-      (effects (font (size 1.27 1.27)))
-    )
-    (property "Footprint" "" (id 2) (at 0 0 0)
-      (effects (font (size 1.27 1.27)) hide)
-    )
-    (property "Datasheet" "" (id 3) (at 0 0 0)
-      (effects (font (size 1.27 1.27)) hide)
-    )
-    (pin "HI")
-    (pin "LI")
-    (pin "HO")
-    (pin "LO")
-    (pin "HS")
-    (pin "VDD")
-    (pin "VSS")
-    (pin "HB")
+    (property "Value" "UCC27211AQDDARQ1" (id 1) (at 45 1337 0)
+      (effects (font (size 1.27 1.27)))
+    )
+    (property "Footprint" "Package_SO:SOIC-8-1EP_3.9x4.9mm_P1.27mm_EP2.95x3.4mm" (id 2) (at 0 0 0)
+      (effects (font (size 1.27 1.27)) hide)
+    )
+    (property "Datasheet" "https://www.ti.com/lit/ds/symlink/ucc27211a-q1.pdf" (id 3) (at 0 0 0)
+      (effects (font (size 1.27 1.27)) hide)
+    )
+    (pin "5")
+    (pin "6")
+    (pin "3")
+    (pin "8")
+    (pin "4")
+    (pin "1")
+    (pin "7")
+    (pin "2")
     (instances
       (project "microgrid_48v"
@@
       (effects (font (size 1.27 1.27)))
     )
-    (property "Value" "UCC27211A" (id 1) (at 157 1337 0)
-      (effects (font (size 1.27 1.27)))
-    )
-    (property "Footprint" "" (id 2) (at 0 0 0)
-      (effects (font (size 1.27 1.27)) hide)
-    )
-    (property "Datasheet" "" (id 3) (at 0 0 0)
-      (effects (font (size 1.27 1.27)) hide)
-    )
-    (pin "HI")
-    (pin "LI")
-    (pin "HO")
-    (pin "LO")
-    (pin "HS")
-    (pin "VDD")
-    (pin "VSS")
-    (pin "HB")
+    (property "Value" "UCC27211AQDDARQ1" (id 1) (at 157 1337 0)
+      (effects (font (size 1.27 1.27)))
+    )
+    (property "Footprint" "Package_SO:SOIC-8-1EP_3.9x4.9mm_P1.27mm_EP2.95x3.4mm" (id 2) (at 0 0 0)
+      (effects (font (size 1.27 1.27)) hide)
+    )
+    (property "Datasheet" "https://www.ti.com/lit/ds/symlink/ucc27211a-q1.pdf" (id 3) (at 0 0 0)
+      (effects (font (size 1.27 1.27)) hide)
+    )
+    (pin "5")
+    (pin "6")
+    (pin "3")
+    (pin "8")
+    (pin "4")
+    (pin "1")
+    (pin "7")
+    (pin "2")
     (instances
       (project "microgrid_48v"
@@
       (effects (font (size 1.27 1.27)))
     )
-    (property "Value" "UCC27211A" (id 1) (at 269 1337 0)
-      (effects (font (size 1.27 1.27)))
-    )
-    (property "Footprint" "" (id 2) (at 0 0 0)
-      (effects (font (size 1.27 1.27)) hide)
-    )
-    (property "Datasheet" "" (id 3) (at 0 0 0)
-      (effects (font (size 1.27 1.27)) hide)
-    )
-    (pin "HI")
-    (pin "LI")
-    (pin "HO")
-    (pin "LO")
-    (pin "HS")
-    (pin "VDD")
-    (pin "VSS")
-    (pin "HB")
+    (property "Value" "UCC27211AQDDARQ1" (id 1) (at 269 1337 0)
+      (effects (font (size 1.27 1.27)))
+    )
+    (property "Footprint" "Package_SO:SOIC-8-1EP_3.9x4.9mm_P1.27mm_EP2.95x3.4mm" (id 2) (at 0 0 0)
+      (effects (font (size 1.27 1.27)) hide)
+    )
+    (property "Datasheet" "https://www.ti.com/lit/ds/symlink/ucc27211a-q1.pdf" (id 3) (at 0 0 0)
+      (effects (font (size 1.27 1.27)) hide)
+    )
+    (pin "5")
+    (pin "6")
+    (pin "3")
+    (pin "8")
+    (pin "4")
+    (pin "1")
+    (pin "7")
+    (pin "2")
     (instances
       (project "microgrid_48v"
@@
       (effects (font (size 1.27 1.27)))
     )
-    (property "Footprint" "" (id 2) (at 0 0 0)
+    (property "Footprint" "Microgrid_48V:DVG0010A_HV" (id 2) (at 0 0 0)
       (effects (font (size 1.27 1.27)) hide)
     )
@@
       (effects (font (size 1.27 1.27)) hide)
     )
-    (pin "IP+")
-    (pin "IP-")
-    (pin "VOUT")
-    (pin "OC")
-    (pin "VS")
-    (pin "GND")
-    (pin "VREF")
-    (pin "VOC")
-    (pin "ALERT")
-    (pin "NC")
+    (pin "1")
+    (pin "2")
+    (pin "6")
+    (pin "7")
+    (pin "8")
+    (pin "3")
+    (pin "5")
+    (pin "9")
+    (pin "4")
+    (pin "10")
     (instances
       (project "microgrid_48v"
@@
       (effects (font (size 1.27 1.27)))
     )
-    (property "Footprint" "" (id 2) (at 0 0 0)
+    (property "Footprint" "Microgrid_48V:DVG0010A_HV" (id 2) (at 0 0 0)
       (effects (font (size 1.27 1.27)) hide)
     )
@@
       (effects (font (size 1.27 1.27)) hide)
     )
-    (pin "IP+")
-    (pin "IP-")
-    (pin "VOUT")
-    (pin "OC")
-    (pin "VS")
-    (pin "GND")
-    (pin "VREF")
-    (pin "VOC")
-    (pin "ALERT")
-    (pin "NC")
+    (pin "1")
+    (pin "2")
+    (pin "6")
+    (pin "7")
+    (pin "8")
+    (pin "3")
+    (pin "5")
+    (pin "9")
+    (pin "4")
+    (pin "10")
     (instances
       (project "microgrid_48v"
@@
       (effects (font (size 1.27 1.27)))
     )
-    (property "Footprint" "" (id 2) (at 0 0 0)
+    (property "Footprint" "Microgrid_48V:DVG0010A_HV" (id 2) (at 0 0 0)
       (effects (font (size 1.27 1.27)) hide)
     )
@@
       (effects (font (size 1.27 1.27)) hide)
     )
-    (pin "IP+")
-    (pin "IP-")
-    (pin "VOUT")
-    (pin "OC")
-    (pin "VS")
-    (pin "GND")
-    (pin "VREF")
-    (pin "VOC")
-    (pin "ALERT")
-    (pin "NC")
-    (instances
-      (project "microgrid_48v"
+    (pin "1")
+    (pin "2")
+    (pin "6")
+    (pin "7")
+    (pin "8")
+    (pin "3")
+    (pin "5")
+    (pin "9")
+    (pin "4")
+    (pin "10")
+    (instances
+      (project "microgrid_48v"
